Commit message: Gazebo sim with standard controller working!

File: description/urdf/6dofexample.urdf.xacro (robot description, xacro)
@@ -6,6 +6,8 @@
   <link name="world"/>
   <xacro:r6bot_description/>
+  <xacro:include filename="gazebo.urdf.xacro"/>
+  <xacro:gazebo controllers="$(find wiimote_teleop)/config/controllers.yaml"/>
   <!-- Import r6bot ros2_control description -->
   <xacro:include filename="$(find wiimote_teleop)/description/urdf/ros2_control.xacro" />
-  <xacro:r6bot_ros2_control name="r6bot"/>
+  <xacro:r6bot_ros2_control name="r6bot" sim="true"/>
 </robot>

File: description/urdf/create_link.xacro (robot description, xacro)
@@ -11,5 +11,5 @@
         <origin xyz="${xyz_offset}" rpy="${rpy_offset}"/>
         <geometry>
-          <mesh filename="package://${mesh_package}/description/meshes/visual/${mesh_name}.dae"/>
+          <mesh filename="$(find ${mesh_package})/description/meshes/visual/${mesh_name}.dae"/>
         </geometry>
       </visual>
@@ -17,5 +17,5 @@
         <origin xyz="${xyz_offset}" rpy="${rpy_offset}"/>
         <geometry>
-          <mesh filename="package://${mesh_package}/description/meshes/collision/${mesh_name}.stl"/>
+          <mesh filename="$(find ${mesh_package})/description/meshes/collision/${mesh_name}.stl"/>
         </geometry>
       </collision>

File: description/urdf/ros2_control.xacro (robot description, xacro)
@@ -1,12 +1,19 @@
 <?xml version="1.0"?>
 <robot xmlns:xacro="http://www.ros.org/wiki/xacro">
-  <xacro:macro name="r6bot_ros2_control" params="name">
+  <xacro:macro name="r6bot_ros2_control" params="name sim">
     <ros2_control name="${name}" type="system">
       <!-- <hardware>
         <plugin>ros2_control_demo_example_7/RobotSystem</plugin>
       </hardware> -->
-      <hardware>
-          <plugin>mock_components/GenericSystem</plugin>
-      </hardware>
+      <xacro:if value="${sim}">
+        <hardware>
+            <plugin>gz_ros2_control/GazeboSimSystem</plugin>
+        </hardware>
+      </xacro:if>
+      <xacro:unless value="${sim}">
+        <hardware>
+            <plugin>mock_components/GenericSystem</plugin>
+        </hardware>
+      </xacro:unless>
       <joint name="joint_1">
         <command_interface name="position">

Commit message: Gripper added!
(Took longer that expected)

File: description/urdf/6dofexample.urdf.xacro (robot description, xacro)
@@ -10,4 +10,6 @@
   <!-- Import r6bot ros2_control description -->
   <xacro:include filename="$(find wiimote_teleop)/description/urdf/ros2_control.xacro" />
-  <xacro:r6bot_ros2_control name="r6bot" sim="true"/>
+  <xacro:r6bot_ros2_control name="r6bot" sim="true" gripper="true"/>
+  <xacro:include filename="$(find wiimote_teleop)/description/urdf/gripper.attach.urdf.xacro"/>
+  <xacro:gripper_attach base="tool0"/>
 </robot>

File: description/urdf/create_link.xacro (robot description, xacro)
@@ -11,5 +11,5 @@
         <origin xyz="${xyz_offset}" rpy="${rpy_offset}"/>
         <geometry>
-          <mesh filename="$(find ${mesh_package})/description/meshes/visual/${mesh_name}.dae"/>
+          <mesh filename="file://$(find ${mesh_package})/description/meshes/visual/${mesh_name}.dae"/>
         </geometry>
       </visual>
@@ -17,5 +17,5 @@
         <origin xyz="${xyz_offset}" rpy="${rpy_offset}"/>
         <geometry>
-          <mesh filename="$(find ${mesh_package})/description/meshes/collision/${mesh_name}.stl"/>
+          <mesh filename="file://$(find ${mesh_package})/description/meshes/collision/${mesh_name}.stl"/>
         </geometry>
       </collision>

File: description/urdf/gripper.urdf.xacro (robot description, xacro)
@@ -1,7 +1,18 @@
 <?xml version="1.0"?>
-<robot xmlns:xacro="http://www.ros.org/wiki/xacro">
-  <xacro:macro name="r6bot_ros2_control" params="name sim gripper:=false">
-    <ros2_control name="${name}" type="system">
-      <xacro:if value="${gripper}">
+<robot name="delto_3f" xmlns:xacro="http://www.ros.org/wiki/xacro">
+    <xacro:include filename="$(find wiimote_teleop)/description/urdf/gripper.links.urdf.xacro" />
+    <link name="tool0" />
+    <joint name="tool0_to_base_fixed" type="fixed">
+        <parent link="tool0" />
+        <child link="base_link_grip" />
+        <origin xyz="0 0 0.1" rpy="0 0 0" />
+    </joint>
+    <ros2_control name="GazeboSimSystem" type="system">
+        <hardware>
+            <plugin>gz_ros2_control/GazeboSimSystem</plugin>
+        </hardware>
+        <hardware>
+            <plugin>mock_components/GenericSystem</plugin>
+        </hardware>
         <!-- Finger 1 joints -->
         <joint name="j_dg_1_1">
@@ -139,111 +150,41 @@
             <state_interface name="effort" />
         </joint>
-      </xacro:if>
-      <!-- <hardware>
-        <plugin>ros2_control_demo_example_7/RobotSystem</plugin>
-      </hardware> -->
-      <xacro:if value="${sim}">
-        <hardware>
-            <plugin>gz_ros2_control/GazeboSimSystem</plugin>
-        </hardware>
-      </xacro:if>
-      <xacro:unless value="${sim}">
-        <hardware>
-            <plugin>mock_components/GenericSystem</plugin>
-        </hardware>
-      </xacro:unless>
-      <joint name="joint_1">
-        <command_interface name="position">
-          <param name="min">${-2*pi}</param>
-          <param name="max">${2*pi}</param>
-        </command_interface>
-        <command_interface name="velocity">
-          <param name="min">-3.15</param>
-          <param name="max">3.15</param>
-        </command_interface>
-        <state_interface name="position">
-          <param name="initial_value">0.0</param>
-        </state_interface>
-        <state_interface name="velocity"/>
-      </joint>
-      <joint name="joint_2">
-        <command_interface name="position">
-          <param name="min">${-2*pi}</param>
-          <param name="max">${2*pi}</param>
-        </command_interface>
-        <command_interface name="velocity">
-          <param name="min">-3.15</param>
-          <param name="max">3.15</param>
-        </command_interface>
-        <state_interface name="position">
-          <param name="initial_value">0.0</param>
-        </state_interface>
-        <state_interface name="velocity"/>
-      </joint>
-      <joint name="joint_3">
-        <command_interface name="position">
-          <param name="min">${-pi}</param>
-          <param name="max">${pi}</param>
-        </command_interface>
-        <command_interface name="velocity">
-          <param name="min">-3.15</param>
-          <param name="max">3.15</param>
-        </command_interface>
-        <state_interface name="position">
-          <param name="initial_value">0.0</param>
-        </state_interface>
-        <state_interface name="velocity"/>
-      </joint>
-      <joint name="joint_4">
-        <command_interface name="position">
-          <param name="min">${-2*pi}</param>
-          <param name="max">${2*pi}</param>
-        </command_interface>
-        <command_interface name="velocity">
-          <param name="min">-3.2</param>
-          <param name="max">3.2</param>
-        </command_interface>
-        <state_interface name="position">
-          <param name="initial_value">0.0</param>
-        </state_interface>
-        <state_interface name="velocity"/>
-      </joint>
-      <joint name="joint_5">
-        <command_interface name="position">
-          <param name="min">${-2*pi}</param>
-          <param name="max">${2*pi}</param>
-        </command_interface>
-        <command_interface name="velocity">
-          <param name="min">-3.2</param>
-          <param name="max">3.2</param>
-        </command_interface>
-        <state_interface name="position">
-          <param name="initial_value">0.0</param>
-        </state_interface>
-        <state_interface name="velocity"/>
-      </joint>
-      <joint name="joint_6">
-        <command_interface name="position">
-          <param name="min">${-2*pi}</param>
-          <param name="max">${2*pi}</param>
-        </command_interface>
-        <command_interface name="velocity">
-          <param name="min">-3.2</param>
-          <param name="max">3.2</param>
-        </command_interface>
-        <state_interface name="position">
-          <param name="initial_value">0.0</param>
-        </state_interface>
-        <state_interface name="velocity"/>
-      </joint>
-      <sensor name="tcp_fts_sensor">
-        <state_interface name="force.x"/>
-        <state_interface name="force.y"/>
-        <state_interface name="force.z"/>
-        <state_interface name="torque.x"/>
-        <state_interface name="torque.y"/>
-        <state_interface name="torque.z"/>
-      </sensor>
     </ros2_control>
-  </xacro:macro>
+    <gazebo>
+        <gravity>false</gravity>
+        <physics type="dart">  <!-- dart 엔진이 일반적으로 더 빠름 -->
+            <max_step_size>0.0</max_step_size>  <!-- 스텝 사이즈 증가 -->
+            <real_time_factor>1.0</real_time_factor>
+            <real_time_update_rate>250</real_time_update_rate>  <!-- 업데이트 레이트 감소 -->
+            <max_contacts>5</max_contacts>  <!-- 접촉점 수 감소 -->
+            <!-- 추가 최적화 설정 -->
+            <solver>
+                <type>quick</type>
+                <iters>10</iters>  <!-- 반복 횟수 감소 -->
+                <precon_iters>0</precon_iters>
+                <sor>1.0</sor>
+            </solver>
+        </physics>
+        <self_collide>0</self_collide>
+        <!-- 렌더링 최적화 -->
+        <visual>
+            <shadows>false</shadows>
+            <grid>false</grid>
+        </visual>
+        <collision_detector>ode</collision_detector>
+        <constraints>
+            <contact_max_correcting_vel>0.0</contact_max_correcting_vel>
+            <cfm>0.0</cfm>
+            <erp>0.0</erp>
+        </constraints>
+        <plugin name="ign_ros2_control::IgnitionROS2ControlPlugin"
+            filename="libign_ros2_control-system.so">
+            <robot_param_node>robot_state_publisher</robot_param_node>
+            <robot_param>robot_description</robot_param>
+            <parameters>$(find dg3f_m_gz)/config/dg3f_m_gz_controller.yaml</parameters>
+            <ros>
+                <namespace>/</namespace>
+            </ros>
+        </plugin>
+    </gazebo>
 </robot>
